File: Ricardo-IgniterBoard/BuckBoost.kicad_sch (KiCad schematic)
At the start: 21 parts, among them Q2 NMOS, U10 TPS55288QRPMRQ1

Commit message: Little touches
Parts:
- added C18, C19: 0.1uF, Capacitor_SMD:C_0402_1005Metric, symbol Device:C_Small
- added C?: 8.2nF, symbol Device:C
- added LED7: RED_LED, LED_SMD:LED_0402_1005Metric, symbol Device:LED_Small
- added R31, R32: 3.3k, Resistor_SMD:R_0402_1005Metric, symbol Device:R_Small
- added R33: 2m, Resistor_SMD:R_2512_6332Metric_Pad1.40x3.35mm_HandSolder, symbol Device:R
- added R34: 3k, Resistor_SMD:R_0402_1005Metric, symbol Device:R_Small
- added R50, R51: 10, Resistor_SMD:R_0402_1005Metric, symbol Device:R_Small
- added R52: 10k, Resistor_SMD:R_0402_1005Metric, symbol Device:R_Small
- added TP3, TP7: TestPoint, TestPoint:TestPoint_Pad_D1.0mm, symbol Connector:TestPoint
- added U7: INA219AxDCN, Package_TO_SOT_SMD:SOT-23-8, symbol Sensor_Energy:INA219AxDCN
- C32: value 15pF -> 6.8pF
- C?: value 4.7nF -> 1nF
- Cin: value 220uF -> 27uF
- Cout: value 33uF -> 47uF
- Coutx: value 10uF -> 15uF
- L?: value 4.7uH -> 2.17uH
- R1: value 383k -> 715k
- R21: value 20k -> 27.4k
- R23: value 10m -> 8.333m
- R?: value 59k -> 237k
Connections:
- net GND: now also C18.2, C?.1, LED7.1 (K), R52.1, U7.3 (GND), U7.7 (A0), U7.8 (A1); no longer U10.28 (DITH/SYNC_2), U10.7 (DITH/SYNC_1)
- net SCL: now also R32.2, TP3.1, U7.5 (SCL)
- net SDA: now also R31.2, TP7.1, U7.6 (SDA)
- net VOUT: now also R33.2, R34.1, R51.1, R52.2
- net VOUT_2: now also R33.1, R50.1
- new net: LED7.2 (A), R34.2
- new net +3V3: C18.1, R31.1, R32.1, U7.4 (VS)
- new net DITH_2: C?.2, U10.28 (DITH/SYNC_2), U10.7 (DITH/SYNC_1)
- new net SHNT_IN+: C19.1, R50.2, U7.1 (IN+)
- new net SHNT_IN-: C19.2, R51.2, U7.2 (IN-)
Other:
- note added: "Didn't change either of these from their source (Crosshair and flint and steel)"
- moved on the sheet: C31, C32, C33, C?, Cin, Cinx, Cout, Coutx, L?, Q2, Q?, R1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
