File: Ricardo-IgniterBoard/BuckBoost.kicad_sch (KiCad schematic)
At the start: 27 parts, among them Q1 NMOS, Q2 NMOS, U10 TPS55288QRPMRQ1

Commit message: Assigning components
And added the thermocouple
Parts:
- Cboot801: renamed from Cboot2; footprint (none) -> Capacitor_SMD:C_0402_1005Metric
- Cboot802: renamed from Cboot1; footprint (none) -> Capacitor_SMD:C_0402_1005Metric
- Ccomp801: renamed from Ccomp2; footprint (none) -> Capacitor_SMD:C_0402_1005Metric
- Ccomp802: renamed from Ccomp; footprint (none) -> Capacitor_SMD:C_0402_1005Metric
- Cdith801: renamed from Cdith; footprint (none) -> Capacitor_SMD:C_0402_1005Metric
- Cin801: renamed from Cin; footprint (none) -> Capacitor_SMD:C_0402_1005Metric
- Cout801: renamed from Cout1; footprint (none) -> Capacitor_SMD:C_0402_1005Metric
- Cout802: renamed from Cout0; footprint (none) -> Capacitor_SMD:C_0402_1005Metric
- Coutx801: renamed from Coutx2; footprint (none) -> Capacitor_SMD:C_0402_1005Metric
- Coutx802: renamed from Coutx1; footprint (none) -> Capacitor_SMD:C_0402_1005Metric
- Coutx803: renamed from Coutx; footprint (none) -> Capacitor_SMD:C_0402_1005Metric
- Cvcc801: renamed from Cvcc; footprint (none) -> Capacitor_SMD:C_0402_1005Metric
- R801: renamed from R1; footprint (none) -> Resistor_SMD:R_0402_1005Metric
- R802: renamed from R2; footprint (none) -> Resistor_SMD:R_0402_1005Metric
- R803: renamed from R19; footprint (none) -> Resistor_SMD:R_0402_1005Metric
- R804: renamed from R28; footprint (none) -> Resistor_SMD:R_0402_1005Metric
- R805: renamed from R29; footprint (none) -> Resistor_SMD:R_0402_1005Metric
- Rcomp801: renamed from Rcomp; footprint (none) -> Resistor_SMD:R_0402_1005Metric
- Rlim801: renamed from Rlim; footprint (none) -> Resistor_SMD:R_0402_1005Metric
- Rsns801: renamed from Rsns; footprint (none) -> Resistor_SMD:R_0402_1005Metric
- renumbered Cinx to Cinx801, L1 to L801, LED7 to LED801, Q1 to Q801, Q2 to Q802, R34 to R806, U10 to U801

Commit message: Assigning footprints
and adding them to layout
Parts:
- L801: footprint (none) -> Inductor_SMD:L_0805_2012Metric
- Q801, Q802: footprint (none) -> iclr:BSZ025N04LS
- U801: footprint iclr:TPS552882QRPMRQ1 -> iclr:CONV_TPS552882QRPMRQ1
Changed lines of the file:
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@@
 			)
 		)
-		(property "Footprint" ""
+		(property "Footprint" "iclr:BSZ025N04LS"
 			(at 118.11 90.17 0)
 			(effects
@@
 			)
 		)
-		(property "Footprint" ""
+		(property "Footprint" "Inductor_SMD:L_0805_2012Metric"
 			(at 195.58 119.38 0)
 			(effects
@@
 			)
 		)
-		(property "Footprint" ""
+		(property "Footprint" "iclr:BSZ025N04LS"
 			(at 93.98 85.09 0)
 			(effects
@@
 			)
 		)
-		(property "Footprint" "iclr:TPS552882QRPMRQ1"
+		(property "Footprint" "iclr:CONV_TPS552882QRPMRQ1"
 			(at 148.59 204.14 0)
 			(effects
